File: schematics_layouts/rev1/kicadproj_pcb/kicadproj.kicad_pcb (KiCad board)
At the start: 2 copper layers, 0 parts

Commit message: Updated PCB layout
Parts:
- added BT1: Battery_header, Connector_PinHeader_2.54mm:PinHeader_1x02_P2.54mm_Vertical, F.Cu at (106.7, 109.2)
- added C1: 100n, Connector_PinHeader_2.54mm:PinHeader_1x03_P2.54mm_Vertical, F.Cu at (147.3, 91.4)
- added C2: 100n, Connector_PinHeader_2.54mm:PinHeader_1x02_P2.54mm_Vertical, F.Cu at (142.2, 111.8)
- added C3: 100u, Connector_PinHeader_2.54mm:PinHeader_1x03_P2.54mm_Vertical, F.Cu at (147.3, 96.5)
- added C4: 100n, Connector_PinHeader_2.54mm:PinHeader_1x02_P2.54mm_Vertical, F.Cu at (144.8, 94.0)
- added C5: 100u, Connector_PinHeader_2.54mm:PinHeader_1x03_P2.54mm_Vertical, F.Cu at (167.6, 116.8)
- added J1: DS3231_board, Connector_PinHeader_2.54mm:PinHeader_1x06_P2.54mm_Vertical, F.Cu at (121.9, 91.4)
- added J2: LM386_board, Connector_PinHeader_2.54mm:PinHeader_1x04_P2.54mm_Vertical, F.Cu at (175.3, 114.3)
- added J3: microSD_board, Connector_PinHeader_2.54mm:PinHeader_1x06_P2.54mm_Vertical, F.Cu at (157.5, 88.9)
- added Q1: Si2323DS_on_TO220, Connector_PinHeader_2.54mm:PinHeader_1x03_P2.54mm_Vertical, F.Cu at (124.5, 114.3)
- added Q2: Si2323DS_on_TO220, Connector_PinHeader_2.54mm:PinHeader_1x03_P2.54mm_Vertical, F.Cu at (104.1, 114.3)
- added R1: 1K, Connector_PinHeader_2.54mm:PinHeader_1x04_P2.54mm_Vertical, F.Cu at (127.0, 124.5)
- added R2: 4K7, Connector_PinHeader_2.54mm:PinHeader_1x04_P2.54mm_Vertical, F.Cu at (137.2, 124.5)
- added SW1: WAKE Switch, Connector_PinHeader_2.54mm:PinHeader_1x03_P2.54mm_Vertical, F.Cu at (132.1, 116.8)
- added SW2: SET 15MIN, Connector_PinHeader_2.54mm:PinHeader_1x03_P2.54mm_Vertical, F.Cu at (152.4, 121.9)
- added U2: ATmega328P-PU, Package_DIP:DIP-28_W7.62mm, F.Cu at (127.0, 106.7)
Routing:
- net GND: track 0.00 -> 272.8 mm, vias 0 -> 16
- net /+BATT: track 0.00 -> 243.8 mm, vias 0 -> 12
- net VCC: track 0.00 -> 83.8 mm, vias 0 -> 4
- net /SLEEP: track 0.00 -> 58.4 mm, vias 0 -> 6
- net Net-(SW2-2): track 0.00 -> 35.6 mm, vias 0 -> 2
- net /VIN: track 0.00 -> 35.6 mm, vias 0 -> 2
- net /MISO: track 0.00 -> 33.0 mm, vias 0 -> 2
- net /SCK: track 0.00 -> 30.5 mm, vias 0 -> 2
- net /MOSI: track 0.00 -> 27.9 mm, vias 0 -> 2
- net unconnected-(U2-Pin_9-Pad9): track 0.00 -> 10.2 mm
- net unconnected-(U2-Pin_6-Pad6): track 0.00 -> 10.2 mm
- net unconnected-(U2-Pin_24-Pad24): track 0.00 -> 10.2 mm
- net unconnected-(U2-Pin_23-Pad23): track 0.00 -> 10.2 mm
- net unconnected-(U2-Pin_2-Pad2): track 0.00 -> 10.2 mm
- net unconnected-(U2-Pin_14-Pad14): track 0.00 -> 10.2 mm
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Other:
- board outline added: 81.3 x 50.8 mm
