File: schematics_layouts/rev1/kicadproj/kicadproj.kicad_sch (KiCad schematic)
At the start: 54 parts, among them Q1 DS3231, Q2 DS3231, SW1 WAKE Switch, SW2 SET 15MIN, SW3 LOUD, SW4 NIGHT, U2 ATmega328P-PU

Commit message: Updated Makefile; Updated wiki page; Fixed PFET names on schematic; Added kicad project for PCB layout
Parts:
- Q1, Q2: value DS3231 -> Si2323DS
Changed lines of the file:
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@@
 			)
 		)
-		(property "Value" "DS3231"
+		(property "Value" "Si2323DS"
 			(at 210.82 36.83 90)
 			(effects
@@
 			)
 		)
-		(property "Value" "DS3231"
+		(property "Value" "Si2323DS"
 			(at 176.53 40.64 0)
 			(effects

Commit message: Revised all docs, removed C5 (never heard about it); Updated wiki with some news
Parts:
- removed C5: 100u, symbol Device:CP
Changed lines of the file:
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@@
 	)
 	(junction
-		(at 63.5 163.83)
-		(diameter 0)
-		(color 0 0 0 0)
-	)
-	(junction
 		(at 41.91 26.67)
 		(diameter 0)
@@
 	)
 	(junction
-		(at 69.85 109.22)
-		(diameter 0)
-		(color 0 0 0 0)
-	)
-	(junction
 		(at 39.37 114.3)
 		(diameter 0)
@@
 	(wire
 		(pts
-			(xy 20.32 130.81) (xy 20.32 109.22)
-		)
-		(stroke
-			(width 0)
-			(type default)
-		)
-	)
-	(wire
-		(pts
 			(xy 256.54 157.48) (xy 252.73 157.48)
 		)
@@
 	(wire
 		(pts
-			(xy 69.85 105.41) (xy 69.85 109.22)
+			(xy 69.85 105.41) (xy 69.85 114.3)
 		)
 		(stroke
@@
 	(wire
 		(pts
-			(xy 20.32 163.83) (xy 63.5 163.83)
-		)
-		(stroke
-			(width 0)
-			(type default)
-		)
-	)
-	(wire
-		(pts
 			(xy 63.5 161.29) (xy 104.14 161.29)
 		)
@@
 	(wire
 		(pts
-			(xy 69.85 109.22) (xy 69.85 114.3)
-		)
-		(stroke
-			(width 0)
-			(type default)
-		)
-	)
-	(wire
-		(pts
 			(xy 146.05 64.77) (xy 146.05 60.96)
 		)
@@
 	(wire
 		(pts
-			(xy 20.32 109.22) (xy 69.85 109.22)
-		)
-		(stroke
-			(width 0)
-			(type default)
-		)
-	)
-	(wire
-		(pts
 			(xy 135.89 41.91) (xy 146.05 41.91)
 		)
@@
 	(wire
 		(pts
-			(xy 20.32 138.43) (xy 20.32 163.83)
-		)
-		(stroke
-			(width 0)
-			(type default)
-		)
-	)
-	(wire
-		(pts
 			(xy 208.28 120.65) (xy 214.63 120.65)
 		)
@@
 	(wire
 		(pts
-			(xy 63.5 166.37) (xy 63.5 163.83)
-		)
-		(stroke
-			(width 0)
-			(type default)
-		)
-	)
-	(wire
-		(pts
-			(xy 63.5 163.83) (xy 63.5 161.29)
+			(xy 63.5 161.29) (xy 63.5 166.37)
 		)
 		(stroke
@@
 					(unit 1)
 				)
-			)
-		)
-	)
-	(symbol
-		(lib_id "Device:CP")
-		(at 20.32 134.62 0)
-		(unit 1)
-		(exclude_from_sim no)
-		(in_bom yes)
-		(on_board yes)
-		(dnp no)
-		(property "Reference" "C5"
-			(at 15.748 130.048 0)
-			(effects
-				(font
-					(size 1.27 1.27)
-				)
-				(justify left)
-			)
-		)
-		(property "Value" "100u"
-			(at 13.97 137.668 0)
-			(effects
-				(font
-					(size 1.27 1.27)
-				)
-				(justify left)
-			)
-		)
-		(property "Footprint" ""
-			(at 21.2852 138.43 0)
-			(effects
-				(font
-					(size 1.27 1.27)
-				)
-				(hide yes)
-			)
-		)
-		(property "Datasheet" "~"
-			(at 20.32 134.62 0)
-			(effects
-				(font
-					(size 1.27 1.27)
-				)
-				(hide yes)
-			)
-		)
-		(property "Description" "Polarized capacitor"
-			(at 20.32 134.62 0)
-			(effects
-				(font
-					(size 1.27 1.27)
-				)
-				(hide yes)
-			)
-		)
-		(pin "1"
-		)
-		(pin "2"
-		)
-		(instances
-			(project "kicadproj"
-				(path "/ca541a5b-595f-4bc9-94a8-fb0af63f5122"
-					(reference "C5")
-					(unit 1)
-				)
