File: schematics_layouts/rev1/kicadproj/kicadproj.kicad_sch (KiCad schematic)
At the start: 49 parts, among them Q1 Si2323DS, Q2 Si2323DS, SW1 WAKE Switch, SW2 SET 15MIN, SW3 LOUD, SW4 NIGHT, U2 ATmega328P-PU

Commit message: Fixed small error on schematic for 1b; updated docs
Parts:
- renumbered R3 to RB2
Changed lines of the file:
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@@
 		(dnp no)
 		(fields_autoplaced yes)
-		(property "Reference" "R3"
+		(property "Reference" "RB2"
 			(at 93.98 124.4599 0)
 			(effects
@@
 			(project "kicadproj"
 				(path "/ca541a5b-595f-4bc9-94a8-fb0af63f5122"
-					(reference "R3")
+					(reference "RB2")
 					(unit 1)
 				)
