File: schematics_layouts/rev1/kicadproj_pcb_rev1b/kicadproj.kicad_pcb (KiCad board)
At the start: 2 copper layers, 86.4 x 50.8 mm, 16 parts, among them J1 DS3231_board, J2 LM386_board, J3 microSD_board, Q1 Si2323DS_on_TO220, Q2 Si2323DS_on_TO220, SW1 WAKE Switch, SW2 SET 15MIN, U2 ATmega328P-PU

Commit message: Revised PCB layouts; Created PCB layout revision 1c; Updated docs
Routing:
- net GND: track 302.3 -> 309.9 mm
- net /+BATT: track 246.4 -> 254.0 mm
Other:
- board size 86.4 x 50.8 mm -> 86.4 x 53.3 mm
- board text added: "1"
- board text added: "4.5V IN"
- board text added: "AUDIO"
- board text added: "GND"
- board text added: "RTC"
- board text added: "SDCARD"
- board text added: "SET 15MIN"
- board text added: "SET HR"
- board text added: "Seikosha80 github.com/comododragon 2024"
Changed lines of the file:
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@@
 	(title_block
 		(title "Seikosha80 Westminster Chimer")
-		(rev "1")
+		(rev "1b")
 		(comment 1 "/kicadproj/output.pdf for discrete schematic")
 		(comment 2 "https://github.com/comododragon/seikosha80/blob/main/schematics_layouts/rev1")
@@
 	)
 	(gr_rect
-		(start 106.68 78.74)
+		(start 106.68 76.2)
 		(end 193.04 129.54)
 		(stroke
@@
 		(layer "Edge.Cuts")
 	)
+	(gr_text "SET 15MIN"
+		(at 152.4 124.46 0)
+		(layer "F.SilkS")
+		(effects
+			(font
+				(size 1 1)
+				(thickness 0.1)
+			)
+		)
+	)
+	(gr_text "4.5V IN"
+		(at 109.22 111.76 0)
+		(layer "F.SilkS")
+		(effects
+			(font
+				(size 1 1)
+				(thickness 0.1)
+			)
+			(justify left)
+		)
+	)
 	(gr_text "This PCB revision\nuses a stripboard\n(hence predefined\ntracks)."
 		(at 195.58 96.52 0)
@@
 		)
 	)
+	(gr_text "GND"
+		(at 170.18 91.44 0)
+		(layer "F.SilkS")
+		(effects
+			(font
+				(size 1 1)
+				(thickness 0.1)
+			)
+		)
+	)
+	(gr_text "GND"
+		(at 134.62 93.98 0)
+		(layer "F.SilkS")
+		(effects
+			(font
+				(size 1 1)
+				(thickness 0.1)
+			)
+		)
+	)
+	(gr_text "RTC"
+		(at 119.38 88.9 0)
+		(layer "F.SilkS")
+		(effects
+			(font
+				(size 1 1)
+				(thickness 0.1)
+			)
+			(justify left)
+		)
+	)
+	(gr_text "SDCARD"
+		(at 154.94 86.36 0)
+		(layer "F.SilkS")
+		(effects
+			(font
+				(size 1 1)
+				(thickness 0.1)
+			)
+			(justify left)
+		)
+	)
+	(gr_text "GND"
+		(at 109.22 116.84 90)
+		(layer "F.SilkS")
+		(effects
+			(font
+				(size 1 1)
+				(thickness 0.1)
+			)
+			(justify left)
+		)
+	)
+	(gr_text "AUDIO"
+		(at 190.5 119.38 0)
+		(layer "F.SilkS")
+		(effects
+			(font
+				(size 1 1)
+				(thickness 0.1)
+			)
+			(justify right)
+		)
+	)
+	(gr_text "GND"
+		(at 180.34 119.38 0)
+		(layer "F.SilkS")
+		(effects
+			(font
+				(size 1 1)
+				(thickness 0.1)
+			)
+		)
+	)
+	(gr_text "Seikosha80\ngithub.com/comododragon\n2024"
+		(at 190.5 78.74 0)
+		(layer "F.SilkS")
+		(effects
+			(font
+				(size 1 1)
+				(thickness 0.1)
+			)
+			(justify right top)
+		)
+	)
+	(gr_text "SET HR"
+		(at 132.08 124.46 0)
+		(layer "F.SilkS")
+		(effects
+			(font
+				(size 1 1)
+				(thickness 0.1)
+			)
+		)
+	)
+	(gr_text "1"
+		(at 127 109.22 90)
+		(layer "F.SilkS")
+		(effects
+			(font
+				(size 1 1)
+				(thickness 0.1)
+			)
+			(justify left)
+		)
+	)
+	(gr_text_box "Rev. 1: Compact PCB\nRev. 1b: Optimised for daughter cards\nRev. 1c: Optimised for buttons placement"
+		(start 208.28 129.54)
+		(end 256.54 144.78)
+		(layer "F.Cu")
+		(effects
+			(font
+				(size 1.5 1.5)
+				(thickness 0.3)
+				(bold yes)
+			)
+			(justify left top)
+		)
+		(border yes)
+		(stroke
+			(width 0.2)
+			(type solid)
+		)
+	)
+	(gr_text_box "Revision"
+		(start 208.28 124.46)
+		(end 256.54 129.54)
+		(layer "F.Cu")
+		(effects
+			(font
+				(size 1.5 1.5)
+				(thickness 0.3)
+				(bold yes)
+			)
+			(justify left top)
+		)
+		(border yes)
+		(stroke
+			(width 0.2)
+			(type solid)
+		)
+	)
 	(segment
 		(start 111.76 121.92)
@@
 	)
 	(segment
-		(start 170.18 109.22)
-		(end 180.34 109.22)
+		(start 134.62 81.28)
+		(end 134.62 88.9)
 		(width 0.2)
 		(layer "F.Cu")
@@
 	)
 	(segment
-		(start 180.34 106.68)
-		(end 182.88 106.68)
+		(start 142.24 81.28)
+		(end 142.24 88.9)
 		(width 0.2)
 		(layer "F.Cu")
@@
 	)
 	(segment
-		(start 170.18 106.68)
-		(end 170.18 99.06)
+		(start 170.18 109.22)
+		(end 180.34 109.22)
 		(width 0.2)
 		(layer "F.Cu")
@@
 	)
 	(segment
-		(start 144.78 116.84)
-		(end 144.78 121.92)
+		(start 180.34 106.68)
+		(end 182.88 106.68)
 		(width 0.2)
 		(layer "F.Cu")
@@
 	)
 	(segment
-		(start 134.62 83.82)
-		(end 134.62 88.9)
+		(start 170.18 106.68)
+		(end 170.18 99.06)
 		(width 0.2)
 		(layer "F.Cu")
@@
 	)
 	(segment
-		(start 111.76 106.68)
-		(end 111.76 83.82)
+		(start 144.78 116.84)
+		(end 144.78 121.92)
 		(width 0.2)
 		(layer "F.Cu")
@@
 	)
 	(segment
-		(start 142.24 83.82)
-		(end 142.24 88.9)
+		(start 111.76 106.68)
+		(end 111.76 81.28)
 		(width 0.2)
 		(layer "F.Cu")
@@
 	)
 	(via
-		(at 142.24 83.82)
+		(at 142.24 81.28)
 		(size 0.6)
 		(drill 0.3)
@@
 	)
 	(via
-		(at 111.76 83.82)
+		(at 111.76 81.28)
 		(size 0.6)
 		(drill 0.3)
@@
 	)
 	(via
-		(at 134.62 83.82)
+		(at 134.62 81.28)
 		(size 0.6)
 		(drill 0.3)
@@
 	)
 	(segment
-		(start 111.76 83.82)
-		(end 187.96 83.82)
+		(start 142.24 99.06)
+		(end 142.24 88.9)
 		(width 2)
 		(layer "B.Cu")
@@
 	)
 	(segment
-		(start 142.24 99.06)
-		(end 142.24 88.9)
+		(start 111.76 81.28)
+		(end 187.96 81.28)
 		(width 2)
 		(layer "B.Cu")
@@
 	)
 	(segment
-		(start 147.32 86.36)
-		(end 147.32 88.9)
+		(start 116.84 111.76)
+		(end 119.38 111.76)
 		(width 0.2)
 		(layer "F.Cu")
@@
 	)
 	(segment
-		(start 116.84 111.76)
-		(end 119.38 111.76)
+		(start 147.32 83.82)
+		(end 147.32 88.9)
 		(width 0.2)
 		(layer "F.Cu")
@@
 	)
 	(segment
-		(start 132.08 86.36)
+		(start 132.08 83.82)
 		(end 132.08 88.9)
 		(width 0.2)
@@
 	(segment
 		(start 116.84 106.68)
-		(end 116.84 86.36)
+		(end 116.84 83.82)
 		(width 0.2)
 		(layer "F.Cu")
@@
 	)
 	(via
-		(at 147.32 86.36)
+		(at 147.32 83.82)
 		(size 0.6)
 		(drill 0.3)
@@
 	)
 	(via
-		(at 132.08 86.36)
+		(at 132.08 83.82)
 		(size 0.6)
 		(drill 0.3)
@@
 	)
 	(via
-		(at 116.84 86.36)
+		(at 116.84 83.82)
 		(size 0.6)
 		(drill 0.3)
@@
 	)
 	(segment
-		(start 187.96 86.36)
-		(end 111.76 86.36)
+		(start 142.24 106.68)
+		(end 142.24 116.84)
 		(width 2)
 		(layer "B.Cu")
@@
 	)
 	(segment
-		(start 142.24 106.68)
-		(end 142.24 116.84)
+		(start 111.76 124.46)
+		(end 187.96 124.46)
 		(width 2)
 		(layer "B.Cu")
@@
 	)
 	(segment
-		(start 111.76 124.46)
-		(end 187.96 124.46)
+		(start 187.96 83.82)
+		(end 111.76 83.82)
 		(width 2)
 		(layer "B.Cu")

Commit message: Revised all docs, removed C5 (never heard about it); Updated wiki with some news
Parts:
- removed C5: 100u, Connector_PinHeader_2.54mm:PinHeader_1x03_P2.54mm_Vertical
Changed lines of the file:
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@@
-		)
-	)
-	(footprint "Connector_PinHeader_2.54mm:PinHeader_1x03_P2.54mm_Vertical"
-		(layer "F.Cu")
-		(at 187.96 111.76 -90)
-		(descr "Through hole straight pin header, 1x03, 2.54mm pitch, single row")
-		(tags "Through hole pin header THT 1x03 2.54mm single row")
-		(property "Reference" "C5"
-			(at 0 -2.33 90)
-			(layer "F.SilkS")
-			(effects
-				(font
-					(size 1 1)
-					(thickness 0.15)
-				)
-			)
-		)
-		(property "Value" "100u"
-			(at 0 7.41 90)
-			(layer "F.Fab")
-			(effects
-				(font
-					(size 1 1)
-					(thickness 0.15)
-				)
-			)
-		)
-		(property "Footprint" "Connector_PinHeader_2.54mm:PinHeader_1x03_P2.54mm_Vertical"
-			(at 0 0 -90)
-			(unlocked yes)
-			(layer "F.Fab")
-			(hide yes)
-			(effects
-				(font
-					(size 1.27 1.27)
-				)
-			)
-		)
-		(property "Datasheet" ""
-			(at 0 0 -90)
-			(unlocked yes)
-			(layer "F.Fab")
-			(hide yes)
-			(effects
-				(font
-					(size 1.27 1.27)
-				)
-			)
-		)
-		(property "Description" "Polarized capacitor"
-			(at 0 0 -90)
-			(unlocked yes)
-			(layer "F.Fab")
-			(hide yes)
-			(effects
-				(font
-					(size 1.27 1.27)
-				)
-			)
-		)
-		(property ki_fp_filters "CP_*")
-		(sheetname "Root")
-		(sheetfile "kicadproj.kicad_sch")
-		(attr through_hole)
-		(fp_line
-			(start -1.33 6.41)
-			(end 1.33 6.41)
-			(stroke
-				(width 0.12)
-				(type solid)
-			)
-			(layer "F.SilkS")
-		)
-		(fp_line
-			(start -1.33 1.27)
-			(end -1.33 6.41)
-			(stroke
-				(width 0.12)
-				(type solid)
-			)
-			(layer "F.SilkS")
-		)
-		(fp_line
-			(start -1.33 1.27)
-			(end 1.33 1.27)
-			(stroke
-				(width 0.12)
-				(type solid)
-			)
-			(layer "F.SilkS")
-		)
-		(fp_line
-			(start 1.33 1.27)
-			(end 1.33 6.41)
-			(stroke
-				(width 0.12)
-				(type solid)
-			)
-			(layer "F.SilkS")
-		)
-		(fp_line
-			(start -1.33 0)
-			(end -1.33 -1.33)
-			(stroke
-				(width 0.12)
-				(type solid)
-			)
-			(layer "F.SilkS")
-		)
-		(fp_line
-			(start -1.33 -1.33)
-			(end 0 -1.33)
-			(stroke
-				(width 0.12)
-				(type solid)
-			)
-			(layer "F.SilkS")
-		)
-		(fp_line
-			(start -1.8 6.85)
-			(end 1.8 6.85)
-			(stroke
-				(width 0.05)
-				(type solid)
-			)
-			(layer "F.CrtYd")
-		)
-		(fp_line
-			(start 1.8 6.85)
-			(end 1.8 -1.8)
-			(stroke
-				(width 0.05)
-				(type solid)
-			)
-			(layer "F.CrtYd")
-		)
-		(fp_line
-			(start -1.8 -1.8)
-			(end -1.8 6.85)
-			(stroke
-				(width 0.05)
-				(type solid)
-			)
-			(layer "F.CrtYd")
-		)
-		(fp_line
-			(start 1.8 -1.8)
-			(end -1.8 -1.8)
-			(stroke
-				(width 0.05)
-				(type solid)
-			)
-			(layer "F.CrtYd")
-		)
-		(fp_line
-			(start -1.27 6.35)
-			(end -1.27 -0.635)
-			(stroke
-				(width 0.1)
-				(type solid)
-			)
-			(layer "F.Fab")
-		)
-		(fp_line
-			(start 1.27 6.35)
-			(end -1.27 6.35)
-			(stroke
-				(width 0.1)
-				(type solid)
-			)
-			(layer "F.Fab")
-		)
-		(fp_line
-			(start -1.27 -0.635)
-			(end -0.635 -1.27)
-			(stroke
-				(width 0.1)
-				(type solid)
-			)
-			(layer "F.Fab")
-		)
-		(fp_line
-			(start -0.635 -1.27)
-			(end 1.27 -1.27)
-			(stroke
-				(width 0.1)
-				(type solid)
-			)
-			(layer "F.Fab")
-		)
-		(fp_line
-			(start 1.27 -1.27)
-			(end 1.27 6.35)
-			(stroke
-				(width 0.1)
-				(type solid)
-			)
-			(layer "F.Fab")
-		)
-		(fp_text user "${REFERENCE}"
-			(at 0 2.54 180)
-			(layer "F.Fab")
-			(effects
-				(font
-					(size 1 1)
-					(thickness 0.15)
-				)
-			)
-		)
-		(pad "1" thru_hole rect
-			(at 0 0 270)
-			(size 1.7 1.7)
-			(drill 1)
-			(layers "*.Cu" "*.Mask")
-			(remove_unused_layers no)
-			(net 4 "VCC")
-			(pintype "passive")
-		)
-		(pad "3" thru_hole oval
-			(at 0 5.08 270)
-			(size 1.7 1.7)
-			(drill 1)
-			(layers "*.Cu" "*.Mask")
-			(remove_unused_layers no)
-			(net 1 "GND")
-			(pintype "passive")
-		)
-		(model "${KISYS3DMOD}/Connector_PinHeader_2.54mm.3dshapes/PinHeader_1x03_P2.54mm_Vertical.wrl"
-			(offset
-				(xyz 0 0 0)
-			)
-			(scale
-				(xyz 1 1 1)
-			)
-			(rotate
-				(xyz 0 0 0)
-			)
 		)
 	)
